File: KiCad/IrrigationController.kicad_sch (KiCad schematic)
At the start: 17 parts, among them J1 Conn_01x09, J2 USB_C_Receptacle, J3 Conn_01x10, SW1 SW_Push, SW2 SW_Push, U1 ESP32-S3-WROOM-2, U2 PCF8574AT, U3 PCF8574AT

Commit message: add ams1117
Parts:
- added J4: Power in, symbol Connector_Generic:Conn_01x02
- added U4: AMS1117-3.3, Package_TO_SOT_SMD:SOT-223-3_TabPin2, symbol Regulator_Linear:AMS1117-3.3
- added U5: AMS1117-5.0, Package_TO_SOT_SMD:SOT-223-3_TabPin2, symbol Regulator_Linear:AMS1117-5.0
- J1: value Conn_01x09 -> Button in
- J3: value Conn_01x10 -> Relay out
Connections:
- net +3.3V: now also U4.2 (VO)
- net +5V: now also U5.2 (VO)
- net GND: now also J4.2 (Pin_2), U4.1 (GND), U5.1 (GND)
- new net +12V: J4.1 (Pin_1), U4.3 (VI), U5.3 (VI)

Commit message: add TPS6213x 3.3v and 5v regulators
Parts:
- added C10, C7: 100n, Capacitor_SMD:C_0805_2012Metric_Pad1.18x1.45mm_HandSolder, symbol Device:C_Small
- added C11, C8: 3.3n, Capacitor_SMD:C_0805_2012Metric_Pad1.18x1.45mm_HandSolder, symbol Device:C_Small
- added C12, C6: 10u, Capacitor_SMD:C_0805_2012Metric_Pad1.18x1.45mm_HandSolder, symbol Device:C_Small
- added C13, C9: 22u, Capacitor_SMD:C_0805_2012Metric_Pad1.18x1.45mm_HandSolder, symbol Device:C_Small
- added L1, L2: 1/2.2u, symbol Device:L
- added R5, R6: 100k, Resistor_SMD:R_0805_2012Metric_Pad1.20x1.40mm_HandSolder, symbol Device:R_Small
- added U6: TPS62132, Package_DFN_QFN:VQFN-16-1EP_3x3mm_P0.5mm_EP1.68x1.68mm_ThermalVias, symbol Regulator_Switching:TPS62132
- added U7: TPS62133, Package_DFN_QFN:VQFN-16-1EP_3x3mm_P0.5mm_EP1.68x1.68mm_ThermalVias, symbol Regulator_Switching:TPS62133
- added U8: TPS62130, Package_DFN_QFN:VQFN-16-1EP_3x3mm_P0.5mm_EP1.68x1.68mm_ThermalVias, symbol Regulator_Switching:TPS62130
- C1: value C_Small -> 10u; footprint (none) -> Capacitor_SMD:C_0805_2012Metric_Pad1.18x1.45mm_HandSolder
- C2, C3, C4, C5: footprint (none) -> Capacitor_SMD:C_0805_2012Metric_Pad1.18x1.45mm_HandSolder
- R1, R2, R3, R4: footprint (none) -> Resistor_SMD:R_0805_2012Metric_Pad1.20x1.40mm_HandSolder
Connections:
- net +12V: now also C10.1, C12.1, C6.1, C7.1, U6.10 (VIN), U6.11 (VIN), U6.12 (VIN), U6.13 (EN), U7.10 (VIN), U7.11 (VIN), U7.12 (VIN), U7.13 (EN)
- net +3.3V: now also C9.1, L1.2, R5.1, U6.14 (VOS)
- net +5V: now also J3.10 (Pin_10), C13.1, L2.2, R6.1, U7.14 (VOS); no longer J3.1 (Pin_1)
- net GND: now also J3.1 (Pin_1), C10.2, C11.2, C12.2, C13.2, C6.2, C7.2, C8.2, C9.2, U6.15 (GND), U6.16 (GND), U6.17 (GND), U6.5 (FB), U6.6 (GND), U6.7 (FSW), U6.8 (DEF), U7.15 (GND), U7.16 (GND), U7.17 (GND), U7.5 (FB), U7.6 (GND), U7.7 (FSW), U7.8 (DEF); no longer J3.10 (Pin_10)
- new net: L2.1, U7.1 (SW), U7.2 (SW), U7.3 (SW)
- new net: R6.2, U7.4 (PG)
- new net: C11.1, U7.9 (SS/TR)
- new net: U8.1 (SW), U8.2 (SW), U8.3 (SW)
- new net: U8.10 (VIN), U8.11 (VIN), U8.12 (VIN)
- new net: U8.15 (GND), U8.16 (GND), U8.17 (GND), U8.6 (GND)
- new net: R5.2, U6.4 (PG)
- new net: L1.1, U6.1 (SW), U6.2 (SW), U6.3 (SW)
- new net: C8.1, U6.9 (SS/TR)
Other:
- company: (none) -> Paulus Handke
- title: (none) -> Irrigation Controller
- moved on the sheet: U4, U5

Commit message: assign footprints
Parts:
- C1, C12, C6: footprint Capacitor_SMD:C_0805_2012Metric_Pad1.18x1.45mm_HandSolder -> Capacitor_SMD:C_1210_3225Metric_Pad1.33x2.70mm_HandSolder
- L1, L2: footprint (none) -> Inductor_SMD:L_APV_ANR4026
Changed lines of the file:
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@@
 			)
 		)
-		(property "Footprint" "Capacitor_SMD:C_0805_2012Metric_Pad1.18x1.45mm_HandSolder"
+		(property "Footprint" "Capacitor_SMD:C_1210_3225Metric_Pad1.33x2.70mm_HandSolder"
 			(at 137.16 148.59 0)
 			(effects
@@
 			)
 		)
-		(property "Footprint" ""
+		(property "Footprint" "Inductor_SMD:L_APV_ANR4026"
 			(at 157.48 161.29 0)
 			(effects
@@
 			)
 		)
-		(property "Footprint" ""
+		(property "Footprint" "Inductor_SMD:L_APV_ANR4026"
 			(at 102.87 161.29 0)
 			(effects
@@
 			)
 		)
-		(property "Footprint" "Capacitor_SMD:C_0805_2012Metric_Pad1.18x1.45mm_HandSolder"
+		(property "Footprint" "Capacitor_SMD:C_1210_3225Metric_Pad1.33x2.70mm_HandSolder"
 			(at 82.55 148.59 0)
 			(effects
@@
 			)
 		)
-		(property "Footprint" "Capacitor_SMD:C_0805_2012Metric_Pad1.18x1.45mm_HandSolder"
+		(property "Footprint" "Capacitor_SMD:C_1210_3225Metric_Pad1.33x2.70mm_HandSolder"
 			(at 83.82 54.61 0)
 			(effects
